File: schematics/aquila_main/aquila_main.sch (KiCad schematic (older format))
At the start: 36 parts, among them IC1 TPS62152, IC2 TPS62132

Commit message: added connections for telemetry radio
Parts:
- added C?: 1u, symbol aquila_main-rescue:C-cusf-kicad
- added C?: 100n, symbol aquila_main-rescue:C-cusf-kicad
- added C?: 100p, symbol aquila_main-rescue:C-cusf-kicad
- added Y?: 30M, symbol Device:Crystal_Small
- C1, C2, C3, C4, C5, C6, C7, C8, C? (x9): symbol cusf-kicad:C -> aquila_main-rescue:C-cusf-kicad
- IC1, IC2: symbol cusf-kicad:TPS62132 -> aquila_main-rescue:TPS62132-cusf-kicad
- L1, L2: symbol cusf-kicad:L -> aquila_main-rescue:L-cusf-kicad
- Q? (x2): symbol cusf-kicad:Si5515CDC -> aquila_main-rescue:Si5515CDC-cusf-kicad
- R1, R2, R3, R? (x3): symbol cusf-kicad:R -> aquila_main-rescue:R-cusf-kicad
Connections:
- net 3v3: now also U?.6 (VDD), U?.8 (VDD), C?.1, C?.1, C?.1
- net GND: now also U?.1 (SDN), C?.2, C?.2, C?.2
- net MISO: now also U?.13 (SDO)
- net MOSI: now also U?.14 (SDI)
- net SCLK: now also U?.12 (SCLK)
- net radio_int: now reaches U?.11 (~IRQ)
- net radio_cs: now reaches U?.15 (~SEL)
- net at U?.16 (XOUT): now also Y?.2
- net at U?.17 (XIN): now also Y?.1
- net radio_rxp: now reaches U?.2 (RXp)
- net radio_rxn: now reaches U?.3 (RXn)
- net radio_tx: now reaches U?.4 (TX)
- no-connect marks 4 -> 9
Other:
- note added: "Telemetry Radio"
- moved on the sheet: U?
