File: schematics/aquila_main/aquila_main.kicad_sch (KiCad schematic)
At the start: 126 parts

Commit message: added order numbers and footprints to small parts
Parts:
- D? (x2): Farnell (none) -> 2317410
- D?: footprint (none) -> aquila:DO-214AA
- D?: footprint (none) -> aquila:DO-214AA; Farnell (none) -> 1797898
- J? (x5): footprint (none) -> aquila:MP_2.54_screw_terminal_2x1; Farnell (none) -> 3817460
- J?: DigiKey (none) -> A99328-ND
- J? (x2): Mouser (none) -> 960-PCB.SMAFST.J.AHT
- J?: footprint (none) -> Connector_PinHeader_2.54mm:PinHeader_1x06_P2.54mm_Vertical
- J? (x2): DigiKey (none) -> 36-1043P-ND
- U?: DigiKey (none) -> 223-1622-1-ND
- U?: DigiKey (none) -> 505-ADXL357BEZ-ND
- U?: DigiKey (none) -> 336-4346-1-ND
- U?: Farnell (none) -> 2383074
- U? (x2): Farnell (none) -> 3008143
- U?: DigiKey (none) -> 495-2363-1-ND
- U?: Mouser (none) -> 873-SKY65723-81
- Y?: footprint (none) -> aquila:crystal_ABM8; Farnell (none) -> 3228351
Changed lines of the file:
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@@
       (effects (font (size 1.27 1.27)) hide)
     )
+    (property "DigiKey" "223-1622-1-ND" (id 4) (at 283.21 91.44 0)
+      (effects (font (size 1.27 1.27)) hide)
+    )
     (pin "10")
     (pin "11")
@@
       (effects (font (size 1.27 1.27)) (justify left))
     )
-    (property "Footprint" "" (id 2) (at 328.93 205.74 0)
+    (property "Footprint" "aquila:MP_2.54_screw_terminal_2x1" (id 2) (at 328.93 205.74 0)
       (effects (font (size 1.27 1.27)) hide)
     )
@@
       (effects (font (size 1.27 1.27)) hide)
     )
+    (property "Farnell" "3817460" (id 4) (at 328.93 205.74 0)
+      (effects (font (size 1.27 1.27)) hide)
+    )
     (pin "1")
     (pin "2")
@@
       (effects (font (size 1.27 1.27)) hide)
     )
+    (property "DigiKey" "505-ADXL357BEZ-ND" (id 4) (at 170.18 67.31 0)
+      (effects (font (size 1.27 1.27)) hide)
+    )
     (pin "1")
     (pin "10")
@@
       (effects (font (size 1.27 1.27)) hide)
     )
+    (property "DigiKey" "336-4346-1-ND" (id 4) (at 86.36 175.26 0)
+      (effects (font (size 1.27 1.27)) hide)
+    )
     (pin "1")
     (pin "10")
@@
       (effects (font (size 1.27 1.27)) hide)
     )
+    (property "DigiKey" "A99328-ND" (id 4) (at 69.85 119.38 0)
+      (effects (font (size 1.27 1.27)) hide)
+    )
     (pin "1")
     (pin "2")
@@
       (effects (font (size 1.27 1.27)) (justify left))
     )
-    (property "Footprint" "" (id 2) (at 269.24 170.18 0)
+    (property "Footprint" "aquila:MP_2.54_screw_terminal_2x1" (id 2) (at 269.24 170.18 0)
       (effects (font (size 1.27 1.27)) hide)
     )
@@
       (effects (font (size 1.27 1.27)) hide)
     )
+    (property "Farnell" "3817460" (id 4) (at 269.24 170.18 0)
+      (effects (font (size 1.27 1.27)) hide)
+    )
     (pin "1")
     (pin "2")
@@
       (effects (font (size 1.27 1.27)) hide)
     )
+    (property "Farnell" "2383074" (id 4) (at 179.07 43.18 0)
+      (effects (font (size 1.27 1.27)) hide)
+    )
     (pin "1")
     (pin "2")
@@
       (effects (font (size 1.27 1.27)) hide)
     )
+    (property "Farnell" "3008143" (id 4) (at 82.55 39.37 0)
+      (effects (font (size 1.27 1.27)) hide)
+    )
     (pin "1")
     (pin "2")
@@
       (effects (font (size 1.27 1.27)) hide)
     )
+    (property "Farnell" "2317410" (id 4) (at 95.25 102.87 90)
+      (effects (font (size 1.27 1.27)) hide)
+    )
     (pin "1")
     (pin "2")
@@
       (effects (font (size 1.27 1.27)) hide)
     )
+    (property "Mouser" "960-PCB.SMAFST.J.AHT" (id 4) (at 203.2 162.56 0)
+      (effects (font (size 1.27 1.27)) hide)
+    )
     (pin "1")
     (pin "2")
@@
       (effects (font (size 1.27 1.27)) (justify left))
     )
-    (property "Footprint" "" (id 2) (at 269.24 205.74 0)
+    (property "Footprint" "aquila:MP_2.54_screw_terminal_2x1" (id 2) (at 269.24 205.74 0)
       (effects (font (size 1.27 1.27)) hide)
     )
@@
       (effects (font (size 1.27 1.27)) hide)
     )
+    (property "Farnell" "3817460" (id 4) (at 269.24 205.74 0)
+      (effects (font (size 1.27 1.27)) hide)
+    )
     (pin "1")
     (pin "2")
@@
       (effects (font (size 1.27 1.27)) (justify left))
     )
-    (property "Footprint" "" (id 2) (at 73.66 170.18 0)
+    (property "Footprint" "aquila:crystal_ABM8" (id 2) (at 73.66 170.18 0)
       (effects (font (size 1.27 1.27)) hide)
     )
-    (property "Datasheet" "~" (id 3) (at 73.66 170.18 0)
+    (property "Datasheet" "https://www.farnell.com/datasheets/2792510.pdf" (id 3) (at 73.66 170.18 0)
+      (effects (font (size 1.27 1.27)) hide)
+    )
+    (property "Farnell" "3228351" (id 4) (at 73.66 170.18 90)
       (effects (font (size 1.27 1.27)) hide)
     )
@@
       (effects (font (size 1.27 1.27)) hide)
     )
+    (property "Mouser" "960-PCB.SMAFST.J.AHT" (id 4) (at 203.2 234.95 0)
+      (effects (font (size 1.27 1.27)) hide)
+    )
     (pin "1")
     (pin "2")
@@
       (effects (font (size 1.27 1.27)) (justify left))
     )
-    (property "Footprint" "" (id 2) (at 158.75 29.21 0)
+    (property "Footprint" "aquila:MP_2.54_screw_terminal_2x1" (id 2) (at 158.75 29.21 0)
       (effects (font (size 1.27 1.27)) hide)
     )
@@
       (effects (font (size 1.27 1.27)) hide)
     )
+    (property "Farnell" "3817460" (id 4) (at 158.75 29.21 90)
+      (effects (font (size 1.27 1.27)) hide)
+    )
     (pin "1")
     (pin "2")
@@
     (property "Reference" "D?" (id 0) (at 196.85 242.57 0))
     (property "Value" "D_TVS" (id 1) (at 196.85 245.11 0))
-    (property "Footprint" "" (id 2) (at 196.85 240.03 0)
+    (property "Footprint" "aquila:DO-214AA" (id 2) (at 196.85 240.03 0)
       (effects (font (size 1.27 1.27)) hide)
     )
-    (property "Datasheet" "" (id 3) (at 196.85 240.03 0)
+    (property "Datasheet" "1797898" (id 3) (at 196.85 240.03 0)
       (effects (font (size 1.27 1.27)) hide)
     )
@@
       (effects (font (size 1.27 1.27)) hide)
     )
+    (property "DigiKey" "495-2363-1-ND" (id 4) (at 127 241.3 0)
+      (effects (font (size 1.27 1.27)) hide)
+    )
     (pin "1")
     (pin "2")
@@
       (effects (font (size 1.27 1.27)) hide)
     )
+    (property "Mouser" "873-SKY65723-81" (id 4) (at 161.29 234.95 0)
+      (effects (font (size 1.27 1.27)) hide)
+    )
     (pin "1")
     (pin "2")
@@
       (effects (font (size 1.27 1.27)) hide)
     )
+    (property "Farnell" "2317410" (id 4) (at 95.25 54.61 90)
+      (effects (font (size 1.27 1.27)) hide)
+    )
     (pin "1")
     (pin "2")
@@
       (effects (font (size 1.27 1.27)) (justify right))
     )
-    (property "Footprint" "" (id 2) (at 204.47 123.19 0)
+    (property "Footprint" "Connector_PinHeader_2.54mm:PinHeader_1x06_P2.54mm_Vertical" (id 2) (at 204.47 123.19 0)
       (effects (font (size 1.27 1.27)) hide)
     )
@@
     (property "Reference" "D?" (id 0) (at 196.85 170.18 0))
     (property "Value" "D_TVS" (id 1) (at 196.85 172.72 0))
-    (property "Footprint" "" (id 2) (at 196.85 167.64 0)
+    (property "Footprint" "aquila:DO-214AA" (id 2) (at 196.85 167.64 0)
       (effects (font (size 1.27 1.27)) hide)
     )
@@
       (effects (font (size 1.27 1.27)) hide)
     )
+    (property "Farnell" "1797898" (id 4) (at 196.85 167.64 0)
+      (effects (font (size 1.27 1.27)) hide)
+    )
     (pin "1")
     (pin "2")
@@
       (effects (font (size 1.27 1.27)) (justify left))
     )
-    (property "Footprint" "" (id 2) (at 328.93 170.18 0)
+    (property "Footprint" "aquila:MP_2.54_screw_terminal_2x1" (id 2) (at 328.93 170.18 0)
       (effects (font (size 1.27 1.27)) hide)
     )
@@
       (effects (font (size 1.27 1.27)) hide)
     )
+    (property "Farnell" "3817460" (id 4) (at 328.93 170.18 0)
+      (effects (font (size 1.27 1.27)) hide)
+    )
     (pin "1")
     (pin "2")
@@
       (effects (font (size 1.27 1.27)) hide)
     )
+    (property "Farnell" "3008143" (id 4) (at 82.55 87.63 0)
+      (effects (font (size 1.27 1.27)) hide)
+    )
     (pin "1")
     (pin "2")
@@
       (effects (font (size 1.27 1.27)) hide)
     )
+    (property "DigiKey" "36-1043P-ND" (id 4) (at 140.97 39.37 0)
+      (effects (font (size 1.27 1.27)) hide)
+    )
     (pin "1")
     (pin "2")
@@
       (effects (font (size 1.27 1.27)) hide)
     )
+    (property "DigiKey" "36-1043P-ND" (id 4) (at 140.97 48.26 0)
+      (effects (font (size 1.27 1.27)) hide)
+    )
     (pin "1")
     (pin "2")
@@
     )
     (path "/777fba89-cb4f-4686-a79e-65cd02296ad1"
-      (reference "D?") (unit 1) (value "D_TVS") (footprint "")
+      (reference "D?") (unit 1) (value "D_TVS") (footprint "aquila:DO-214AA")
     )
     (path "/9ce76768-9f86-44d1-bfc9-4078dbfad525"
@@
     )
     (path "/d90a6c10-3ef9-46d4-8d0c-ee65981220b9"
-      (reference "D?") (unit 1) (value "D_TVS") (footprint "")
+      (reference "D?") (unit 1) (value "D_TVS") (footprint "aquila:DO-214AA")
     )
     (path "/041540dd-66e6-44c5-9d56-d11d2216d19d"
@@
     )
     (path "/00000000-0000-0000-0000-000062227685"
-      (reference "J?") (unit 1) (value "PYRO_4") (footprint "")
+      (reference "J?") (unit 1) (value "PYRO_4") (footprint "aquila:MP_2.54_screw_terminal_2x1")
     )
     (path "/00000000-0000-0000-0000-0000626a7bfd"
@@
     )
     (path "/1565b66f-a0cb-4bf4-ac0f-80784d58f1c3"
-      (reference "J?") (unit 1) (value "PYRO_1") (footprint "")
+      (reference "J?") (unit 1) (value "PYRO_1") (footprint "aquila:MP_2.54_screw_terminal_2x1")
     )
     (path "/4110da84-f44d-44bf-a7e1-605bbfbf191a"
@@
     )
     (path "/41b1a2de-e58a-452f-a200-68f659f67a89"
-      (reference "J?") (unit 1) (value "PYRO_3") (footprint "")
+      (reference "J?") (unit 1) (value "PYRO_3") (footprint "aquila:MP_2.54_screw_terminal_2x1")
     )
     (path "/558e1c63-e133-4ecd-9417-018852123092"
@@
     )
     (path "/66f82d02-ed0c-47ac-9270-d9bbe0e47982"
-      (reference "J?") (unit 1) (value "PWR") (footprint "")
+      (reference "J?") (unit 1) (value "PWR") (footprint "aquila:MP_2.54_screw_terminal_2x1")
     )
     (path "/99c1f101-5d22-400f-9743-bb2f2b4a649e"
@@
     )
     (path "/d2a2af03-5cef-466b-b6f2-22346d252541"
-      (reference "J?") (unit 1) (value "BARO") (footprint "")
+      (reference "J?") (unit 1) (value "BARO") (footprint "Connector_PinHeader_2.54mm:PinHeader_1x06_P2.54mm_Vertical")
     )
     (path "/e686095d-0490-4c28-9dd6-8c7ca208b053"
-      (reference "J?") (unit 1) (value "PYRO_2") (footprint "")
+      (reference "J?") (unit 1) (value "PYRO_2") (footprint "aquila:MP_2.54_screw_terminal_2x1")
     )
     (path "/f5d2d9c4-79f5-4d67-94a1-36a8c64f3985"
@@
     )
     (path "/5261fde7-e5b4-4565-991d-43c69ff8ae8d"
-      (reference "Y?") (unit 1) (value "30M") (footprint "")
+      (reference "Y?") (unit 1) (value "30M") (footprint "aquila:crystal_ABM8")
     )
   )

Commit message: changed pyro power to 5V
Parts:
- removed J?: PYRO_4, aquila:MP_2.54_screw_terminal_2x1, symbol Connector:Screw_Terminal_01x02
- removed J?: PYRO_3, aquila:MP_2.54_screw_terminal_2x1, symbol Connector:Screw_Terminal_01x02
- removed J?: PYRO_2, aquila:MP_2.54_screw_terminal_2x1, symbol Connector:Screw_Terminal_01x02
- removed Q? (x6): IRF7509PbF, aquila:IRF7509PbF, symbol aquila:IRF7509PbF
- removed R? (x6): 10k, symbol aquila:R-cusf-kicad
- removed R? (x3): 100k, symbol aquila:R-cusf-kicad
- added J?: PYRO_4, aquila:MP_2.54_screw_terminal_2x1, symbol Connector:Screw_Terminal_01x02
- added J?: PYRO_3, aquila:MP_2.54_screw_terminal_2x1, symbol Connector:Screw_Terminal_01x02
- added J?: PYRO_2, aquila:MP_2.54_screw_terminal_2x1, symbol Connector:Screw_Terminal_01x02
- added Q? (x6): IRF7509PbF, aquila:IRF7509PbF, symbol aquila:IRF7509PbF
- added R? (x7): 100k, symbol aquila:R-cusf-kicad
- added R? (x6): 10k, symbol aquila:R-cusf-kicad
- added R? (x4): 200k, symbol aquila:R-cusf-kicad
- J?: footprint Connector_PinHeader_2.54mm:PinHeader_1x06_P2.54mm_Vertical -> aquila:molex_nano_fit_x6_105310-1106; Farnell (none) -> 2820682
- L?: value 68u -> 100u
- R?: value 100 -> 330
- U?: value LM2576S-3.3/NOPB -> LM2576D2TR4-5G; Farnell 3008143 -> 2534166
Connections:
- net GND: now also J?.2 (Pin_2), J?.2 (Pin_2), J?.2 (Pin_2), Q?.1 (S1), Q?.1 (S1), Q?.1 (S1), R?.2, R?.2, R?.2, R?.2, R?.2, R?.2, R?.2
- net pyro_ch2: now also Q?.2 (G1), R?.1
- net pyro_ch3: now also Q?.2 (G1), R?.1
- net pyro_ch4: now also Q?.2 (G1), R?.1
- net pyro_cont1: now also R?.1, R?.2; no longer J?.1 (Pin_1), Q?.5 (D2), Q?.6 (D2), R?.2
- net pyro_cont2: now also R?.1, R?.2
- net pyro_cont3: now also R?.1, R?.2
- net pyro_cont4: now also R?.1, R?.2
- net pyro_pwr: now also Q?.3 (S2), Q?.3 (S2), Q?.3 (S2), R?.1, R?.1, R?.1, R?.1, R?.1, R?.1
- new net: J?.1 (Pin_1), Q?.5 (D2), Q?.6 (D2), R?.1, R?.2 (x4)
- new net: Q?.4 (G2), Q?.7 (D1), Q?.8 (D1), R?.2 (x3)
Other:
- note added: "3A, 5V for Pyrotechnics"
- note removed: "3A, 3.3V for Pyrotechnics"
- note removed: "Pyro channel 2"
- note removed: "Pyro channel 3"
- note removed: "Pyro channel 4"
- moved on the sheet: R?

Commit message: added connector for servos
Parts:
- added J?: SERVO, aquila:molex_nano_fit_x6_105310-1106, symbol Connector:Conn_01x06_Male
Connections:
- net GND: now also J?.1 (Pin_1)
- net pyro_sply: now also J?.6 (Pin_6)
- net servo_2: now reaches U?.10 (8_TX2_IN1)
- net servo_2: now also J?.4 (Pin_4)
- net servo_3: now reaches U?.11 (9_OUT1C)
- net servo_3: now also J?.3 (Pin_3)
- net servo_4: now reaches U?.12 (10_CS_MQSR)
- net servo_4: now also J?.2 (Pin_2)
- net servo_1: now reaches U?.9 (7_RX2_OUT1A)
- net servo_1: now also J?.5 (Pin_5)
- no-connect marks 51 -> 47
Other:
- note added: "Servo Connector"
Changed lines of the file:
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@@
   (no_connect (at 154.94 87.63))
   (no_connect (at 139.7 128.27))
-  (no_connect (at 255.27 57.15))
   (no_connect (at 311.15 44.45))
   (no_connect (at 311.15 46.99))
@@
   (no_connect (at 311.15 106.68))
   (no_connect (at 311.15 114.3))
-  (no_connect (at 255.27 59.69))
-  (no_connect (at 255.27 62.23))
-  (no_connect (at 255.27 64.77))
   (no_connect (at 373.38 175.26))
   (no_connect (at 68.58 227.33))
@@
     (stroke (width 0) (type default) (color 0 0 0 0))
   )
+  (wire (pts (xy 254 64.77) (xy 255.27 64.77))
+    (stroke (width 0) (type default) (color 0 0 0 0))
+  )
   (wire (pts (xy 143.51 234.95) (xy 144.78 234.95))
     (stroke (width 0) (type default) (color 0 0 0 0))
@@
     (stroke (width 0) (type default) (color 0 0 0 0))
   )
+  (wire (pts (xy 377.19 125.73) (xy 377.19 127))
+    (stroke (width 0) (type default) (color 0 0 0 0))
+  )
   (wire (pts (xy 95.25 106.68) (xy 102.87 106.68))
     (stroke (width 0) (type default) (color 0 0 0 0))
@@
     (stroke (width 0) (type default) (color 0 0 0 0))
   )
+  (wire (pts (xy 375.92 120.65) (xy 379.73 120.65))
+    (stroke (width 0) (type default) (color 0 0 0 0))
+  )
   (wire (pts (xy 264.16 161.29) (xy 261.62 161.29))
     (stroke (width 0) (type default) (color 0 0 0 0))
@@
     (stroke (width 0) (type default) (color 0 0 0 0))
   )
+  (wire (pts (xy 238.76 62.23) (xy 255.27 62.23))
+    (stroke (width 0) (type default) (color 0 0 0 0))
+  )
   (wire (pts (xy 181.61 97.79) (xy 185.42 97.79))
     (stroke (width 0) (type default) (color 0 0 0 0))
@@
     (stroke (width 0) (type default) (color 0 0 0 0))
   )
+  (wire (pts (xy 238.76 57.15) (xy 255.27 57.15))
+    (stroke (width 0) (type default) (color 0 0 0 0))
+  )
   (bus (pts (xy 60.96 227.33) (xy 60.96 229.87))
     (stroke (width 0) (type default) (color 0 0 0 0))
@@
     (stroke (width 0) (type default) (color 0 0 0 0))
   )
+  (polyline (pts (xy 351.79 135.89) (xy 351.79 104.14))
+    (stroke (width 0) (type default) (color 0 0 0 0))
+  )
   (wire (pts (xy 152.4 214.63) (xy 152.4 215.9))
     (stroke (width 0) (type default) (color 0 0 0 0))
@@
     (stroke (width 0) (type default) (color 0 0 0 0))
   )
+  (polyline (pts (xy 398.78 135.89) (xy 351.79 135.89))
+    (stroke (width 0) (type default) (color 0 0 0 0))
+  )
   (wire (pts (xy 156.21 167.64) (xy 156.21 168.91))
     (stroke (width 0) (type default) (color 0 0 0 0))
@@
     (stroke (width 0) (type default) (color 0 0 0 0))
   )
+  (polyline (pts (xy 398.78 104.14) (xy 398.78 135.89))
+    (stroke (width 0) (type default) (color 0 0 0 0))
+  )
   (polyline (pts (xy 281.94 181.61) (xy 223.52 181.61))
     (stroke (width 0) (type default) (color 0 0 0 0))
@@
     (stroke (width 0) (type default) (color 0 0 0 0))
   )
+  (wire (pts (xy 375.92 115.57) (xy 379.73 115.57))
+    (stroke (width 0) (type default) (color 0 0 0 0))
+  )
   (wire (pts (xy 63.5 234.95) (xy 68.58 234.95))
     (stroke (width 0) (type default) (color 0 0 0 0))
@@
     (stroke (width 0) (type default) (color 0 0 0 0))
   )
+  (wire (pts (xy 375.92 118.11) (xy 379.73 118.11))
+    (stroke (width 0) (type default) (color 0 0 0 0))
+  )
   (wire (pts (xy 184.15 234.95) (xy 185.42 234.95))
     (stroke (width 0) (type default) (color 0 0 0 0))
@@
     (stroke (width 0) (type default) (color 0 0 0 0))
   )
+  (wire (pts (xy 375.92 123.19) (xy 379.73 123.19))
+    (stroke (width 0) (type default) (color 0 0 0 0))
+  )
   (bus (pts (xy 321.31 67.31) (xy 326.39 67.31))
     (stroke (width 0) (type default) (color 0 0 0 0))
@@
     (stroke (width 0) (type default) (color 0 0 0 0))
   )
+  (wire (pts (xy 379.73 125.73) (xy 377.19 125.73))
+    (stroke (width 0) (type default) (color 0 0 0 0))
+  )
   (wire (pts (xy 302.26 187.96) (xy 302.26 189.23))
     (stroke (width 0) (type default) (color 0 0 0 0))
@@
     (stroke (width 0) (type default) (color 0 0 0 0))
   )
+  (wire (pts (xy 238.76 59.69) (xy 255.27 59.69))
+    (stroke (width 0) (type default) (color 0 0 0 0))
+  )
   (wire (pts (xy 185.42 99.06) (xy 189.23 99.06))
     (stroke (width 0) (type default) (color 0 0 0 0))
@@
     (stroke (width 0) (type default) (color 0 0 0 0))
   )
+  (wire (pts (xy 375.92 113.03) (xy 379.73 113.03))
+    (stroke (width 0) (type default) (color 0 0 0 0))
+  )
   (wire (pts (xy 76.2 172.72) (xy 73.66 172.72))
     (stroke (width 0) (type default) (color 0 0 0 0))
@@
     (stroke (width 0) (type default) (color 0 0 0 0))
   )
+  (polyline (pts (xy 351.79 104.14) (xy 398.78 104.14))
+    (stroke (width 0) (type default) (color 0 0 0 0))
+  )
   (wire (pts (xy 68.58 214.63) (xy 68.58 213.36))
     (stroke (width 0) (type default) (color 0 0 0 0))
@@
     (effects (font (size 1.27 1.27)) (justify left bottom))
   )
+  (text "Servo Connector\n" (at 382.27 134.62 0)
+    (effects (font (size 1.27 1.27)) (justify left bottom))
+  )
   (text "3A, 5V  for Pyrotechnics" (at 92.71 115.57 0)
     (effects (font (size 1.27 1.27)) (justify left bottom))
@@
     (effects (font (size 1.27 1.27)) (justify left bottom))
   )
+  (label "servo_1" (at 238.76 57.15 180)
+    (effects (font (size 1.27 1.27)) (justify right bottom))
+  )
   (label "bckp_batt" (at 271.78 124.46 180)
     (effects (font (size 1.27 1.27)) (justify right bottom))
@@
     (effects (font (size 1.27 1.27)) (justify left bottom))
   )
+  (label "servo_4" (at 375.92 123.19 180)
+    (effects (font (size 1.27 1.27)) (justify right bottom))
+  )
   (label "SCLK1" (at 312.42 69.85 0)
     (effects (font (size 1.27 1.27)) (justify left bottom))
@@
     (effects (font (size 1.27 1.27)) (justify right bottom))
   )
+  (label "pyro_sply" (at 375.92 113.03 180)
+    (effects (font (size 1.27 1.27)) (justify right bottom))
+  )
   (label "pyro_ch4" (at 326.39 92.71 0)
     (effects (font (size 1.27 1.27)) (justify left bottom))
@@
     (effects (font (size 1.27 1.27)) (justify right bottom))
   )
+  (label "servo_2" (at 238.76 59.69 180)
+    (effects (font (size 1.27 1.27)) (justify right bottom))
+  )
   (label "pyro_ch3" (at 326.39 90.17 0)
     (effects (font (size 1.27 1.27)) (justify left bottom))
@@
     (effects (font (size 1.27 1.27)) (justify right bottom))
   )
+  (label "servo_1" (at 375.92 115.57 180)
+    (effects (font (size 1.27 1.27)) (justify right bottom))
+  )
   (label "SPI1" (at 326.39 67.31 0)
     (effects (font (size 1.27 1.27)) (justify left bottom))
@@
     (effects (font (size 1.27 1.27)) (justify left bottom))
   )
+  (label "servo_3" (at 238.76 62.23 180)
+    (effects (font (size 1.27 1.27)) (justify right bottom))
+  )
   (label "MISO1" (at 247.65 69.85 0)
     (effects (font (size 1.27 1.27)) (justify left bottom))
@@
     (effects (font (size 1.27 1.27)) (justify left bottom))
   )
+  (label "servo_2" (at 375.92 118.11 180)
+    (effects (font (size 1.27 1.27)) (justify right bottom))
+  )
   (label "pyro_pwr" (at 233.68 184.15 180)
     (effects (font (size 1.27 1.27)) (justify right bottom))
@@
     (effects (font (size 1.27 1.27)) (justify right bottom))
   )
+  (label "servo_3" (at 375.92 120.65 180)
+    (effects (font (size 1.27 1.27)) (justify right bottom))
+  )
+  (label "servo_4" (at 254 64.77 180)
+    (effects (font (size 1.27 1.27)) (justify right bottom))
+  )
   (label "radio_int" (at 238.76 87.63 180)
     (effects (font (size 1.27 1.27)) (justify right bottom))
@@
     (pin "1")
   )
+  (symbol (lib_id "power:GND") (at 377.19 127 0) (unit 1)
+    (in_bom yes) (on_board yes)
+    (property "Reference" "#PWR?" (id 0) (at 377.19 133.35 0)
+      (effects (font (size 1.27 1.27)) hide)
+    )
+    (property "Value" "GND" (id 1) (at 377.317 131.3942 0))
+    (property "Footprint" "" (id 2) (at 377.19 127 0)
+      (effects (font (size 1.27 1.27)) hide)
+    )
+    (property "Datasheet" "" (id 3) (at 377.19 127 0)
+      (effects (font (size 1.27 1.27)) hide)
+    )
+    (pin "1")
+  )
   (symbol (lib_id "power:GND") (at 107.95 242.57 0) (unit 1)
     (in_bom yes) (on_board yes)
@@
     (pin "1")
   )
+  (symbol (lib_id "Connector:Conn_01x06_Male") (at 384.81 120.65 180) (unit 1)
+    (in_bom yes) (on_board yes)
+    (property "Reference" "J?" (id 0) (at 386.08 116.84 0)
+      (effects (font (size 1.27 1.27)) (justify right))
+    )
+    (property "Value" "SERVO" (id 1) (at 386.08 119.38 0)
+      (effects (font (size 1.27 1.27)) (justify right))
+    )
+    (property "Footprint" "aquila:molex_nano_fit_x6_105310-1106" (id 2) (at 384.81 120.65 0)
+      (effects (font (size 1.27 1.27)) hide)
+    )
+    (property "Datasheet" "https://www.molex.com/pdm_docs/sd/1053101106_sd.pdf" (id 3) (at 384.81 120.65 0)
+      (effects (font (size 1.27 1.27)) hide)
+    )
+    (property "Farnell" "2820682" (id 5) (at 384.81 120.65 0)
+      (effects (font (size 1.27 1.27)) hide)
+    )
+    (pin "1")
+    (pin "2")
+    (pin "3")
+    (pin "4")
+    (pin "5")
+    (pin "6")
+  )
   (symbol (lib_id "aquila:R-cusf-kicad") (at 327.66 194.31 270) (unit 1)
     (in_bom yes) (on_board yes)
@@
       (reference "#PWR?") (unit 1) (value "GND") (footprint "")
     )
+    (path "/6b06efb6-04cd-4391-898f-4b2fd745e57d"
+      (reference "#PWR?") (unit 1) (value "GND") (footprint "")
+    )
     (path "/74fa530a-bf62-4b88-a3fd-1cc7ee0ae642"
       (reference "#PWR?") (unit 1) (value "GND") (footprint "")
@@
       (reference "J?") (unit 1) (value "PYRO_2") (footprint "aquila:MP_2.54_screw_terminal_2x1")
     )
+    (path "/eee9c670-90b8-4762-9a30-7de865e7ad0f"
+      (reference "J?") (unit 1) (value "SERVO") (footprint "aquila:molex_nano_fit_x6_105310-1106")
+    )
     (path "/f5d2d9c4-79f5-4d67-94a1-36a8c64f3985"
